Commit message: add realsende obstacle avodiance

File: uvbot_description/urdf/uvbot_description.urdf (robot description, URDF)
Before this commit: robot uvbot_description, 6 links, 5 joints
Links:
- added link sonar1_link, mass 0.0258112064800094; collision mesh filename=package://uvbot_description/meshes/sonar1_link.STL; visual mesh filename=package://uvbot_description/meshes/sonar1_link.STL
- added link sonar2_link, mass 0.0258112064800093; collision mesh filename=package://uvbot_description/meshes/sonar2_link.STL; visual mesh filename=package://uvbot_description/meshes/sonar2_link.STL
- added link sonar3_link, mass 0.025811; collision mesh filename=package://uvbot_description/meshes/sonar3_link.STL; visual mesh filename=package://uvbot_description/meshes/sonar3_link.STL
- added link sonar4_link, mass 0; collision mesh filename=package://uvbot_description/meshes/sonar4_link.STL; visual mesh filename=package://uvbot_description/meshes/sonar4_link.STL
- link laser_link: mass 0.26216 -> 0.262164963511652
- link realsense_link: mass 0 -> 0.0449411298420615
- link rightwheel_link: mass 1.419 -> 1.41903797649423
Joints:
- added joint sonar1_joint: type fixed, parent base_link, child sonar1_link, origin xyz=0.15797 0.27578 0.034144 rpy=0.00022064 -0.00047429 1.1354, axis 0 0 0
- added joint sonar2_joint: type fixed, parent base_link, child sonar2_link, origin xyz=0.29939 0.1086 0.034057 rpy=0.00050515 -0.00013585 0.26271, axis 0 0 0
- added joint sonar3_joint: type fixed, parent base_link, child sonar3_link, origin xyz=0.29958 -0.10761 0.033944 rpy=0.0005054 0.00013493 -0.26089, axis 0 0 0
- added joint sonar4_joint: type fixed, parent base_link, child sonar4_link, origin xyz=0.158473613809801 -0.27504791684719 0.0338560706421803 rpy=0.000221499778446617 0.000473886325860837 -1.1335579299033, axis 0 0 0
- joint realsense_joint: origin xyz=0.29721 0.00024774 0.090317 rpy=1.0472 0.0010462 1.5708 -> xyz=0.29721 0.00024774 0.090317 rpy=-0.001208 -0.5236 0.00060402
